File: hardware/IOT/lampatra.sch (KiCad schematic (older format))
At the start: 7 parts

Commit message: Add files via upload
Parts:
- removed J?: Conn_02x04_Row_Letter_First, symbol Conn_02x04_Row_Letter_First
- added C1, C3, C6, C7, C8: 100N, Capacitors_SMD:C_0805_HandSoldering, symbol C
- added J1: Conn_01x02, Pin_Headers:Pin_Header_Straight_1x02_Pitch2.54mm, symbol Conn_01x02
- added J2: Conn_02x04_Top_Bottom, Pin_Headers:Pin_Header_Straight_2x04_Pitch2.54mm, symbol Conn_02x04_Top_Bottom
- added J3, J4: Conn_01x03, Pin_Headers:Pin_Header_Straight_1x03_Pitch2.54mm, symbol Conn_01x03
- added R1: 4K7, Resistors_SMD:R_0805_HandSoldering, symbol R
- added SW1: SW_Push_SPDT, Buttons_Switches_SMD:SW_SPDT_PCM12, symbol SW_Push_SPDT
- added U1, U2, U3, U4: WS2812B, LEDs:LED_WS2812B-PLCC4, symbol WS2812B
- C2, C4: renamed from C?; footprint (none) -> Capacitors_THT:CP_Radial_D4.0mm_P1.50mm
- C5: renamed from C?; footprint (none) -> Capacitors_SMD:C_0805_HandSoldering
- U5: renamed from U?; footprint (none) -> LEDs:LED_WS2812B-PLCC4
- U6: renamed from U?; footprint (none) -> Pin_Headers:Pin_Header_Straight_1x04_Pitch2.54mm; symbol DHT11 -> DHT11-RESCUE-lampatra
- U7: renamed from U?; footprint (none) -> TO_SOT_Packages_SMD:SOT-223
Connections:
- net +3V3: now also U6.1 (vcc), J2.5 (Pin_5), R1.1, SW1.1 (A)
- net +5V: now also U5.1 (VDD), C1.1, C3.1, C6.1, C7.1, C8.1, J1.1 (Pin_1), J3.2 (Pin_2), J4.2 (Pin_2), U1.1 (VDD), U2.1 (VDD), U3.1 (VDD), U4.1 (VDD)
- net GND: now also U5.3 (VSS), U6.4 (gnd), C1.2, C3.2, C6.2, C7.2, C8.2, J1.2 (Pin_2), J2.4 (Pin_4), J3.3 (Pin_3), J4.3 (Pin_3), SW1.3 (C), U1.3 (VSS), U2.3 (VSS), U3.3 (VSS), U4.3 (VSS)
- net at U5.4 (DIN): now also U4.2 (DOUT)
- net GPIO_2: now reaches U6.2 (data)
- net GPIO_2: now also J2.3 (Pin_3), R1.2
- new net: U3.2 (DOUT), U4.4 (DIN)
- new net: U2.2 (DOUT), U3.4 (DIN)
- new net: U1.2 (DOUT), U2.4 (DIN)
- new net CH_PD: J2.7 (Pin_7), SW1.2 (B)
- new net GPIO_0: J2.2 (Pin_2), U1.4 (DIN)
- new net RX: J2.1 (Pin_1), J3.1 (Pin_1)
- new net Rreset: J2.6 (Pin_6)
- new net TX: J2.8 (Pin_8), J4.1 (Pin_1)
- no-connect marks 0 -> 2
Other:
- moved on the sheet: C2, C4, C5, U5, U6, U7
